File: QUANT-01/pcb/quant_v1.sch (EAGLE design)
At the start: 67 parts, among them SW1 SUBMINI_SPDT, SW2 SUBMINI_SPDT, SW3 SUBMINI_SPDT, SW4 SUBMINI_SPDT, SW5_MODE SUBMINI_SPDT, U3 MCP6002, U4 TL074_

Commit message: starting wiring. completed layout of components.
Parts:
- removed C1: 0.33uF, SparkFun-Capacitors:10NF-PTH-10MM-10000V-1-%
- removed C2: 0.1uF, SparkFun-Capacitors:10NF-PTH-10MM-10000V-1-%
- removed TL7805: R-78E5.0-1.0, SparkFun-IC-Power:R-78E5.0-1.0
- added TOUCH_I, TOUCH_II, TOUCH_III, TOUCH_IV, TOUCH_V, TOUCH_VI, TOUCH_VII: (no value), ESSY:TOUCH_PAD_ESSY
- added TOUCH_VIII: touch_8, ESSY:TOUCH_PAD_ESSY
- added U$1, U$2: (no value), ESSY:TOUCH_PAD_INCREMENT
- J3, J4: device SparkFun-Connectors:CONN_09 -> SparkFun-Connectors:CONN_14
Connections:
- removed net GLIDE_WIPER: U4B.-IN, U4B.OUT, VR1.E, VR1.S
- new net GLIDE_3: J3.11, U4B.-IN, U4B.OUT
- new net N$26: J4.8, R8.2
- new net N$33: J4.7, R7.2
- new net N$35: J4.6, R6.2
- new net N$36: J4.5, R5.2
- new net N$40: J4.4, R4.2
- new net N$41: J4.3, R3.2
- new net N$42: J4.2, R2.2
- new net N$43: J4.1, R1.2
- new net N$44: J1.2, TOUCH_I.IN
- new net N$45: J1.3, TOUCH_II.IN
- new net N$46: J1.4, TOUCH_III.IN
- new net N$47: J1.5, TOUCH_IV.IN
- new net N$48: J1.6, TOUCH_V.IN
- new net N$49: J1.7, TOUCH_VI.IN
- new net N$50: J1.8, TOUCH_VII.IN
- new net N$51: J1.9, TOUCH_VIII.IN
- new net N$52: J1.10, U$2.P$1
- new net N$53: J1.11, U$1.P$1
- new net TO_GLIDE_1: J4.10, VR1.A
- new net TO_GLIDE_3: J4.11, VR1.E, VR1.S
- net +12V: no longer C1.1, TL7805.IN
- net 5V: no longer C2.1, TL7805.OUT
- net GLIDE_1: now also J3.10; no longer VR1.A
- net GND: no longer C1.2, C2.2, TL7805.GND
- net LED_I: no longer J4.1, R1.2
- net LED_II: no longer J4.2, R2.2
- net LED_III: no longer J4.3, R3.2
- net LED_IV: no longer J4.4, R4.2
- net LED_V: no longer J4.5, R5.2
- net LED_VI: no longer J4.6, R6.2
- net LED_VII: no longer J4.7, R7.2
- net LED_VIII: no longer J4.8, R8.2
- net TOUCH0: no longer J1.2
- net TOUCH1: no longer J1.3
- net TOUCH10: no longer J1.12
- net TOUCH11: no longer J1.13
- net TOUCH2: no longer J1.4
- net TOUCH3: no longer J1.5
- net TOUCH4: no longer J1.6
- net TOUCH5: no longer J1.7
- net TOUCH6: no longer J1.8
- net TOUCH7: no longer J1.9
- net TOUCH8: no longer J1.10
- net TOUCH9: no longer J1.11
Other:
- moved on the sheet: C5, J1, J2, MCP4725, U4B, U4C, VR1
